Commit message: Added geometry tag

File: husky_description/urdf/decorations.urdf.xacro (robot description, xacro)
@@ -94,4 +94,5 @@
            <geometry>
             <mesh filename="package://husky_description/meshes/dual_arm_bulkhead.dae" />
+           </geometry>
         </collision>
         <inertial>

Commit message: Additional UR5 fixes which make it work

File: husky_description/urdf/decorations.urdf.xacro (robot description, xacro)
@@ -37,5 +37,5 @@
       <child link="top_chassis_link" />
     </joint>
-    <xacro:if value="$(optenv HUSKY_USER_RAILS true)">
+    <xacro:if value="$(optenv HUSKY_USER_RAILS false)">
 	    <!-- Spawn user rails -->
 	    <link name="user_rail_link">
@@ -81,7 +81,7 @@
       <child link="rear_bumper_link" />
     </joint>
-    <xacro:if value="$(optenv DUAL_ARM_BULKHEAD false)">
+    <xacro:if value="$(optenv DUAL_ARM_BULKHEAD true)">
         <!-- Spawn the bulkhead -->
-      <link name="dual_arm_bulkhead_link">
+        <link name="dual_arm_bulkhead_link">
         <visual>
           <origin xyz="0 0 0" rpy="0 0 0" />
@@ -94,12 +94,12 @@
            <geometry>
             <mesh filename="package://husky_description/meshes/dual_arm_bulkhead.dae" />
-           </geometry>
+          </geometry>
         </collision>
-        <inertial>
-          <mass value="9.832"/>
-          <origin xyz="0 0 0" />
-          <inertia ixx="0.177184" ixy="-0.0045887" ixz="0.003812" iyy="0.752238" iyz="0.004194" izz="0.1376" />
-        </inertial>
-      </link>
+          <inertial>
+            <mass value="9.832"/>
+            <origin xyz="0 0 0" />
+            <inertia ixx="0.177184" ixy="-0.0045887" ixz="0.003812" iyy="0.752238" iyz="0.004194" izz="0.1376" />
+          </inertial>
+        </link>
       <!-- Attach bulkhead -->
       <joint name="dual_arm_bulkhead_joint" type="fixed">
@@ -109,5 +109,5 @@
       </joint>
     </xacro:if>
-    <xacro:if value="$(optenv HUSKY_TOP_PLATE_ENABLED true)">
+    <xacro:if value="$(optenv HUSKY_TOP_PLATE_ENABLED false)">
       <!-- Spawn the top plate -->
       <link name="top_plate_link">

File: husky_description/urdf/description.xacro (robot description, xacro)
@@ -22,5 +22,5 @@
 -->
 <robot name="husky" xmlns:xacro="http://ros.org/wiki/xacro">
-  <xacro:arg name="dual_ur5_enabled" default="$(optenv HUSKY_DUAL_UR5_ENABLED false)" />
+  <xacro:arg name="dual_ur5_enabled" default="$(optenv HUSKY_DUAL_UR5_ENABLED true)" />
   <xacro:arg name="laser_enabled" default="false" />
   <xacro:arg name="ur5_enabled" default="false" />

File: husky_description/urdf/dual_arm_husky.urdf.xacro (robot description, xacro)
@@ -1,3 +1,11 @@
 <?xml version="1.0" ?>
+<!-- =================================================================================== -->
+<!-- |    This document was autogenerated by xacro from dual_arm_husky.urdf.xacro      | -->
+<!-- |    EDITING THIS FILE BY HAND IS NOT RECOMMENDED                                 | -->
+<!-- =================================================================================== -->
+<!-- =================================================================================== -->
+<!-- |    This document was autogenerated by xacro from description.xacro              | -->
+<!-- |    EDITING THIS FILE BY HAND IS NOT RECOMMENDED                                 | -->
+<!-- =================================================================================== -->
 <!--
 Software License Agreement (BSD)
@@ -92,7 +100,7 @@
   <link name="inertial_link">
     <inertial>
-      <mass value="48.39054"/>
+      <mass value="0.39054"/>
       <origin xyz="-0.0648 -0.00059 0.07895"/>
-      <inertia ixx="2.1634275613800003" ixy="-0.055452352110000006" ixz="-0.41083822026" iyy="3.5314689495400002" iyz="-0.004366145530000001" izz="4.4759585875" />
+      <inertia ixx="0.001634275613800003" ixy="-0.0055452352110000006" ixz="-0.041083822026" iyy="0.05314689495400002" iyz="-0.0004366145530000001" izz="-0.004759585875"/>
     </inertial>
   </link>
@@ -477,5 +485,6 @@
   <!-- Connect PTU to Husky bulkhead -->
   <joint name="husky_ptu_joint" type="fixed">
-    <origin rpy="0 0 0" xyz="0.345 0.010414 0.19876"/><!-- x-translation still needs to be measured -->
+    <origin rpy="0 0 0" xyz="0.345 0.010414 0.19876"/>
+    <!-- x-translation still needs to be measured -->
     <parent link="dual_arm_bulkhead_link"/>
     <child link="husky_ptu_base_link"/>
@@ -1061,6 +1070,6 @@
             <samples>720</samples>
             <resolution>1</resolution>
-            <min_angle>-2.35619</min_angle>
-            <max_angle>2.35619</max_angle>
+            <min_angle>-3.14</min_angle>
+            <max_angle>3.14</max_angle>
           </horizontal>
         </scan>

File: husky_description/urdf/husky.urdf.xacro (robot description, xacro)
@@ -78,5 +78,5 @@
       <inertial>
         <mass value="46.034"/>
-        <origin xyz="-0.08748 -0.00085 0.09947" />
+        <origin xyz="-0.00065 -0.085 0.062" />
         <inertia ixx="0.6022" ixy="-0.02364" ixz="-0.1197" iyy="1.7386" iyz="-0.001544" izz="2.0296" />
       </inertial>
@@ -111,5 +111,5 @@
     </xacro:husky_wheel>
     <xacro:husky_decorate />
-    <xacro:if value="$(optenv FLIR_PTU_ENABLED false)">
+    <xacro:if value="$(optenv FLIR_PTU_ENABLED true)">
           <xacro:ptu_d46 name="husky_ptu"/>
           <!-- Connect PTU to Husky bulkhead -->
@@ -120,5 +120,5 @@
          </joint>
     </xacro:if>
-    <xacro:if value="$(optenv HUSKY_DUAL_UR5_ENABLED false)">
+    <xacro:if value="$(optenv HUSKY_DUAL_UR5_ENABLED true)">
         <xacro:ur5_robot prefix="l_ur5_arm_" joint_limited="true"/>
         <xacro:ur5_robot prefix="r_ur5_arm_" joint_limited="true"/>
@@ -145,5 +145,5 @@
            <origin xyz="0 0 0" rpy="0 1.57 0"/>
         </xacro:robotiq_fts300>
-        <xacro:if value="$(optenv ROBOTIQ_GRIPPERS_ENABLED false)">
+        <xacro:if value="$(optenv ROBOTIQ_GRIPPERS_ENABLED true)">
             <xacro:robotiq_hand prefix="l_" reflect="1" parent="l_robotiq_fts300_fts_toolside">
                 <origin xyz="0 0 0.08" rpy="1.57 0 0"/>
