Commit message: Separated FT support for grippers. Added bounding box

File: husky_description/urdf/description.xacro (robot description, xacro)
@@ -26,6 +26,47 @@
   <xacro:arg name="ur5_enabled" default="false" />
   <xacro:arg name="kinect_enabled" default="false" />
-  <xacro:arg name="robotiq_grippers_enabled" default="$(optenv ROBOTIQ_GRIPPERS_ENABLED false)" />
-  <xacro:include filename="$(find husky_description)/urdf/dual_arm_husky.urdf.xacro" />
+  <xacro:arg name="robotiq_grippers_enabled" default="$(optenv ROBOTIQ_GRIPPERS_ENABLED true)" />
+  <xacro:include filename="$(find husky_description)/urdf/husky.urdf.xacro" />
   <xacro:husky_robot />
+  <!-- Collision prevention boxes to prevent hitting the cables -->
+  <link name="l_gripper_protection_box">
+    <visual>
+      <origin xyz="0 0 0" rpy="0 0 0" />
+      <geometry>
+        <box size="0.18 0.10 0.07" rpy="0 0 0" />
+      </geometry>
+    </visual>
+    <collision>
+      <origin xyz="0 0 0" rpy="0 0 0" />
+      <geometry>
+        <box size="0.18 0.10 0.07" />
+      </geometry>
+    </collision>
+  </link>
+  <!-- Collision prevention boxes to prevent hitting the cables -->
+  <link name="r_gripper_protection_box">
+    <visual>
+      <origin xyz="0 0 0" rpy="0 0 0" />
+      <geometry>
+        <box size="0.18 0.10 0.07" rpy="0 0 0" />
+      </geometry>
+    </visual>
+    <collision>
+      <origin xyz="0 0 0" rpy="0 0 0" />
+      <geometry>
+        <box size="0.18 0.10 0.07" />
+      </geometry>
+    </collision>
+  </link>
+  <joint name="l_gripper_protection" type="fixed">
+    <parent link="l_robotiq_hand" />
+    <child link="l_gripper_protection_box" />
+    <origin xyz="0 0 0" rpy="0 0 0" />
+  </joint>
+  <!-- Attach the boxes to the gripper to prevent collisions -->
+  <joint name="r_gripper_protection" type="fixed">
+    <parent link="r_robotiq_hand" />
+    <child link="r_gripper_protection_box" />
+    <origin xyz="0 0 0" rpy="0 0 0" />
+  </joint>
 </robot>

File: husky_description/urdf/husky.urdf.xacro (robot description, xacro)
@@ -138,19 +138,27 @@
            <child link="bumblebee2" />
         </joint>
-        <!-- Add force torque model FT300 -->
-        <xacro:robotiq_fts300 parent="l_ur5_arm_ee_link" prefix="l_robotiq_fts300_">
-           <origin xyz="0 0 0" rpy="0 1.57 0"/>
-        </xacro:robotiq_fts300>
-        <xacro:robotiq_fts300 parent="r_ur5_arm_ee_link" prefix="r_robotiq_fts300_">
-           <origin xyz="0 0 0" rpy="0 1.57 0"/>
-        </xacro:robotiq_fts300>
-        <xacro:if value="$(optenv ROBOTIQ_GRIPPERS_ENABLED true)">
-            <xacro:robotiq_hand prefix="l_" reflect="1" parent="l_robotiq_fts300_fts_toolside">
-                <origin xyz="0 0 0.08" rpy="1.57 0 0"/>
-            </xacro:robotiq_hand>
-            <xacro:robotiq_hand prefix="r_" reflect="1" parent="r_robotiq_fts300_fts_toolside">
-                <origin xyz="0 0 0.08" rpy="1.57 0 0"/>
-            </xacro:robotiq_hand>
-        </xacro:if>
+       <xacro:if value="$(optenv ROBOTIQ_GRIPPERS_WITH_FT_ENABLED false)">
+            <!-- Add force torque model FT300 -->
+            <xacro:robotiq_fts300 parent="l_ur5_arm_ee_link" prefix="l_robotiq_fts300_">
+               <origin xyz="0 0 0" rpy="0 1.57 0"/>
+            </xacro:robotiq_fts300>
+            <xacro:robotiq_fts300 parent="r_ur5_arm_ee_link" prefix="r_robotiq_fts300_">
+               <origin xyz="0 0 0" rpy="0 1.57 0"/>
+            </xacro:robotiq_fts300>
+              <xacro:robotiq_hand prefix="l_" reflect="1" parent="l_robotiq_fts300_toolside">
+                 <origin xyz="0 0 0.08" rpy="1.57 0 0"/>
+              </xacro:robotiq_hand>
+              <xacro:robotiq_hand prefix="r_" reflect="1" parent="r_robotiq_fts300_toolside">
+                 <origin xyz="0 0 0.08" rpy="1.57 0 0"/>
+              </xacro:robotiq_hand>
+       </xacro:if>
+       <xacro:if value="$(optenv ROBOTIQ_GRIPPERS_ENABLED true)">
+              <xacro:robotiq_hand prefix="l_" reflect="1" parent="l_ur5_arm_ee_link">
+                 <origin xyz="0.05 0 0" rpy="1.57 1.57 0"/>
+              </xacro:robotiq_hand>
+              <xacro:robotiq_hand prefix="r_" reflect="1" parent="r_ur5_arm_ee_link">
+                 <origin xyz="0.05 0 0" rpy="1.57 1.57 0"/>
+              </xacro:robotiq_hand>
+       </xacro:if>
         <!-- Join left arm to top plate -->
         <joint name="r_ur5_arm_base" type="fixed">
@@ -166,35 +174,4 @@
         </joint>
     </xacro:if>
-    <xacro:if value="$(arg ur5_enabled)">
-      <xacro:property name="reflect" value="-1" />
-      <!-- Spawn arm -->
-      <xacro:ur5_robot prefix="ur5_arm_" joint_limited="true"/>
-      <!-- Join arm -->
-      <joint name="ur5_arm_base" type="fixed">
-        <parent link="top_plate_link" />
-        <child link="ur5_arm_base_link" />
-        <origin xyz="0.3058 0 0.0065" rpy="0.0 0.0 -1.57" />
-      </joint>
-    </xacro:if>
-    <xacro:if value="$(optenv HUSKY_LASER_ENABLED false)">
-      <sick_lms1xx_mount prefix="base" topic="scan"/>
-      <joint name="laser_mount_joint" type="fixed">
-        <origin xyz="$(optenv HUSKY_LMS1XX_XYZ 0.2206 0.0 0.00635)"
-                rpy="$(optenv HUSKY_LMS1XX_RPY 0.0 0.0 0.0)" />
-        <parent link="$(optenv HUSKY_LASER_PARENT_LINK top_plate_link)" />
-        <child link="base_laser_mount" />
-      </joint>
-    </xacro:if>
-    <xacro:if value="$(arg kinect_enabled)">
-      <xacro:sensor_arch prefix="" parent="top_plate_link">
-        <origin xyz="-0.35 0 0.51" rpy="0 0 -3.14"/>
-      </xacro:sensor_arch>
-      <joint name="kinect_frame_joint" type="fixed">
-        <origin xyz="$(optenv HUSKY_KINECT_XYZ 0 0 0)" rpy="$(optenv HUSKY_KINECT_RPY 0 0.18 3.14)" />
-        <parent link="sensor_arch_mount_link"/>
-        <child link="camera_link"/>
-      </joint>
-      <xacro:kinect_camera prefix="camera"/>
-    </xacro:if>
   </xacro:macro>
 </robot>

Commit message: Fixed so it uses palm instead of hand. Also fixed so the sim can use the included box

File: husky_description/urdf/description.xacro (robot description, xacro)
@@ -29,44 +29,3 @@
   <xacro:include filename="$(find husky_description)/urdf/husky.urdf.xacro" />
   <xacro:husky_robot />
-  <!-- Collision prevention boxes to prevent hitting the cables -->
-  <link name="l_gripper_protection_box">
-    <visual>
-      <origin xyz="0 0 0" rpy="0 0 0" />
-      <geometry>
-        <box size="0.18 0.10 0.07" rpy="0 0 0" />
-      </geometry>
-    </visual>
-    <collision>
-      <origin xyz="0 0 0" rpy="0 0 0" />
-      <geometry>
-        <box size="0.18 0.10 0.07" />
-      </geometry>
-    </collision>
-  </link>
-  <!-- Collision prevention boxes to prevent hitting the cables -->
-  <link name="r_gripper_protection_box">
-    <visual>
-      <origin xyz="0 0 0" rpy="0 0 0" />
-      <geometry>
-        <box size="0.18 0.10 0.07" rpy="0 0 0" />
-      </geometry>
-    </visual>
-    <collision>
-      <origin xyz="0 0 0" rpy="0 0 0" />
-      <geometry>
-        <box size="0.18 0.10 0.07" />
-      </geometry>
-    </collision>
-  </link>
-  <joint name="l_gripper_protection" type="fixed">
-    <parent link="l_robotiq_hand" />
-    <child link="l_gripper_protection_box" />
-    <origin xyz="0 0 0" rpy="0 0 0" />
-  </joint>
-  <!-- Attach the boxes to the gripper to prevent collisions -->
-  <joint name="r_gripper_protection" type="fixed">
-    <parent link="r_robotiq_hand" />
-    <child link="r_gripper_protection_box" />
-    <origin xyz="0 0 0" rpy="0 0 0" />
-  </joint>
 </robot>

File: husky_description/urdf/husky.urdf.xacro (robot description, xacro)
@@ -175,3 +175,44 @@
     </xacro:if>
   </xacro:macro>
+   <!-- Collision prevention boxes to prevent hitting the cables -->
+  <link name="l_gripper_protection_box">
+    <visual>
+      <origin xyz="0 0 0" rpy="0 0 0" />
+      <geometry>
+        <box size="0.18 0.10 0.07" rpy="0 0 0" />
+      </geometry>
+    </visual>
+    <collision>
+      <origin xyz="0 0 0.40" rpy="0 0 0" />
+      <geometry>
+        <box size="0.18 0.10 0.07" />
+      </geometry>
+    </collision>
+  </link>
+  <!-- Collision prevention boxes to prevent hitting the cables -->
+  <link name="r_gripper_protection_box">
+    <visual>
+      <origin xyz="0 0 0" rpy="0 0 0" />
+      <geometry>
+        <box size="0.18 0.10 0.07" rpy="0 0 0" />
+      </geometry>
+    </visual>
+    <collision>
+      <origin xyz="0 0 0.40" rpy="0 0 0" />
+      <geometry>
+        <box size="0.18 0.10 0.07" />
+      </geometry>
+    </collision>
+  </link>
+  <joint name="l_gripper_protection" type="fixed">
+    <parent link="l_palm" />
+    <child link="l_gripper_protection_box" />
+    <origin xyz="0 0 0" rpy="0 0 0" />
+  </joint>
+  <!-- Attach the boxes to the gripper to prevent collisions -->
+  <joint name="r_gripper_protection" type="fixed">
+    <parent link="r_palm" />
+    <child link="r_gripper_protection_box" />
+    <origin xyz="0 0 0" rpy="0 0 0" />
+  </joint>
 </robot>
