Commit message: Resolve merge conflicts

File: husky_description/urdf/husky.urdf.xacro (robot description, xacro)
@@ -74,17 +74,9 @@
       <child link="base_footprint" />
     </joint>
-<<<<<<< HEAD
     <!-- Interial link stores the robot's inertial information -->
     <link name="inertial_link">
       <inertial>
         <mass value="46.034"/>
-        <origin xyz="-0.00065 -0.085 0.062" />
-=======
-    <!-- Interial link stores the robot's inertial information
-    <link name="inertial_link">
-      <inertial>
-        <mass value="" />
         <origin xyz="-0.08748 -0.00085 0.09947" />
->>>>>>> 685a629... Shits broken
         <inertia ixx="0.6022" ixy="-0.02364" ixz="-0.1197" iyy="1.7386" iyz="-0.001544" izz="2.0296" />
       </inertial>
@@ -94,9 +86,5 @@
       <parent link="base_link" />
       <child link="inertial_link" />
-<<<<<<< HEAD
     </joint>
-=======
-    </joint> -->
->>>>>>> 685a629... Shits broken
     <!-- IMU Link is the standard mounting position for the UM6 IMU.-->
     <!-- Can be modified with environment variables in /etc/ros/setup.bash -->

Commit message: Added complete bounding box

File: husky_description/urdf/husky.urdf.xacro (robot description, xacro)
@@ -178,13 +178,13 @@
   <link name="l_gripper_protection_box">
     <visual>
-      <origin xyz="0 0 0" rpy="0 0 0" />
-      <geometry>
-        <box size="0.18 0.10 0.07" rpy="0 0 0" />
+      <origin xyz="0.04 0 0" rpy="0 0 0" />
+      <geometry>
+        <box size="0.09 0.10 0.07" rpy="0 0 0" />
       </geometry>
     </visual>
     <collision>
-      <origin xyz="0 0 0.40" rpy="0 0 0" />
-      <geometry>
-        <box size="0.18 0.10 0.07" />
+      <origin xyz="0.04 0 0" rpy="0 0 0" />
+      <geometry>
+        <box size="0.09 0.10 0.07" />
       </geometry>
     </collision>
@@ -193,13 +193,13 @@
   <link name="r_gripper_protection_box">
     <visual>
-      <origin xyz="0 0 0" rpy="0 0 0" />
-      <geometry>
-        <box size="0.18 0.10 0.07" rpy="0 0 0" />
+      <origin xyz="0.04 0 0" rpy="0 0 0" />
+      <geometry>
+        <box size="0.09 0.10 0.07" rpy="0 0 0" />
       </geometry>
     </visual>
     <collision>
-      <origin xyz="0 0 0.40" rpy="0 0 0" />
-      <geometry>
-        <box size="0.18 0.10 0.07" />
+      <origin xyz="0.04 0 0" rpy="0 0 0" />
+      <geometry>
+        <box size="0.09 0.10 0.07" />
       </geometry>
     </collision>

Commit message: Fix imu position

File: husky_description/urdf/husky.urdf.xacro (robot description, xacro)
@@ -91,5 +91,5 @@
     <link name="imu_link"/>
     <joint name="imu_joint" type="fixed">
-      <origin xyz="$(optenv HUSKY_IMU_XYZ 0.19 0 0.149)" rpy="$(optenv HUSKY_IMU_RPY 0 -1.5708 3.1416)" />
+      <origin xyz="$(optenv HUSKY_IMU_XYZ 0.11 0 0.424)" rpy="$(optenv HUSKY_IMU_RPY 0 0 0)" />
       <parent link="base_link" />
       <child link="imu_link" />
