Commit message: change all .dae file to .stl file

File: husky_description/urdf/dual_arm_husky.urdf.xacro (robot description, xacro)
@@ -82,5 +82,5 @@
       <origin rpy="0 0 0" xyz="0 0 0"/>
       <geometry>
-        <mesh filename="package://husky_description/meshes/base_link.dae"/>
+        <mesh filename="package://husky_description/meshes/base_link.stl"/>
       </geometry>
     </visual>
@@ -139,5 +139,5 @@
       <origin rpy="0 0 0" xyz="0 0 0"/>
       <geometry>
-        <mesh filename="package://husky_description/meshes/wheel.dae"/>
+        <mesh filename="package://husky_description/meshes/wheel.stl"/>
       </geometry>
     </visual>
@@ -180,5 +180,5 @@
       <origin rpy="0 0 0" xyz="0 0 0"/>
       <geometry>
-        <mesh filename="package://husky_description/meshes/wheel.dae"/>
+        <mesh filename="package://husky_description/meshes/wheel.stl"/>
       </geometry>
     </visual>
@@ -221,5 +221,5 @@
       <origin rpy="0 0 0" xyz="0 0 0"/>
       <geometry>
-        <mesh filename="package://husky_description/meshes/wheel.dae"/>
+        <mesh filename="package://husky_description/meshes/wheel.stl"/>
       </geometry>
     </visual>
@@ -262,5 +262,5 @@
       <origin rpy="0 0 0" xyz="0 0 0"/>
       <geometry>
-        <mesh filename="package://husky_description/meshes/wheel.dae"/>
+        <mesh filename="package://husky_description/meshes/wheel.stl"/>
       </geometry>
     </visual>
@@ -299,5 +299,5 @@
       <origin rpy="0 0 0" xyz="0 0 0"/>
       <geometry>
-        <mesh filename="package://husky_description/meshes/top_chassis.dae"/>
+        <mesh filename="package://husky_description/meshes/top_chassis.stl"/>
       </geometry>
     </visual>
@@ -312,5 +312,5 @@
     <visual>
       <geometry>
-        <mesh filename="package://husky_description/meshes/bumper.dae"/>
+        <mesh filename="package://husky_description/meshes/bumper.stl"/>
       </geometry>
     </visual>
@@ -326,5 +326,5 @@
     <visual>
       <geometry>
-        <mesh filename="package://husky_description/meshes/bumper.dae"/>
+        <mesh filename="package://husky_description/meshes/bumper.stl"/>
       </geometry>
     </visual>
@@ -341,11 +341,11 @@
       <origin rpy="0 0 0" xyz="0 0 0"/>
       <geometry>
-        <mesh filename="package://husky_description/meshes/dual_arm_bulkhead.dae"/>
-      </geometry>
-    </visual>
-    <collision>
-      <origin rpy="0 0 0" xyz="0 0 0"/>
-      <geometry>
-        <mesh filename="package://husky_description/meshes/dual_arm_bulkhead.dae"/>
+        <mesh filename="package://husky_description/meshes/dual_arm_bulkhead.stl"/>
+      </geometry>
+    </visual>
+    <collision>
+      <origin rpy="0 0 0" xyz="0 0 0"/>
+      <geometry>
+        <mesh filename="package://husky_description/meshes/dual_arm_bulkhead.stl"/>
       </geometry>
     </collision>
@@ -501,5 +501,5 @@
     <visual>
       <geometry>
-        <mesh filename="package://ur_description/meshes/ur5/visual/base.dae"/>
+        <mesh filename="package://ur_description/meshes/ur5/visual/base.stl"/>
       </geometry>
       <material name="LightGrey">
@@ -529,5 +529,5 @@
     <visual>
       <geometry>
-        <mesh filename="package://ur_description/meshes/ur5/visual/shoulder.dae"/>
+        <mesh filename="package://ur_description/meshes/ur5/visual/shoulder.stl"/>
       </geometry>
       <material name="LightGrey">
@@ -557,5 +557,5 @@
     <visual>
       <geometry>
-        <mesh filename="package://ur_description/meshes/ur5/visual/upperarm.dae"/>
+        <mesh filename="package://ur_description/meshes/ur5/visual/upperarm.stl"/>
       </geometry>
       <material name="LightGrey">
@@ -585,5 +585,5 @@
     <visual>
       <geometry>
-        <mesh filename="package://ur_description/meshes/ur5/visual/forearm.dae"/>
+        <mesh filename="package://ur_description/meshes/ur5/visual/forearm.stl"/>
       </geometry>
       <material name="LightGrey">
@@ -613,5 +613,5 @@
     <visual>
       <geometry>
-        <mesh filename="package://ur_description/meshes/ur5/visual/wrist1.dae"/>
+        <mesh filename="package://ur_description/meshes/ur5/visual/wrist1.stl"/>
       </geometry>
       <material name="LightGrey">
@@ -641,5 +641,5 @@
     <visual>
       <geometry>
-        <mesh filename="package://ur_description/meshes/ur5/visual/wrist2.dae"/>
+        <mesh filename="package://ur_description/meshes/ur5/visual/wrist2.stl"/>
       </geometry>
       <material name="LightGrey">
@@ -669,5 +669,5 @@
     <visual>
       <geometry>
-        <mesh filename="package://ur_description/meshes/ur5/visual/wrist3.dae"/>
+        <mesh filename="package://ur_description/meshes/ur5/visual/wrist3.stl"/>
       </geometry>
       <material name="LightGrey">
@@ -775,5 +775,5 @@
     <visual>
       <geometry>
-        <mesh filename="package://ur_description/meshes/ur5/visual/base.dae"/>
+        <mesh filename="package://ur_description/meshes/ur5/visual/base.stl"/>
       </geometry>
       <material name="LightGrey">
@@ -803,5 +803,5 @@
     <visual>
       <geometry>
-        <mesh filename="package://ur_description/meshes/ur5/visual/shoulder.dae"/>
+        <mesh filename="package://ur_description/meshes/ur5/visual/shoulder.stl"/>
       </geometry>
       <material name="LightGrey">
@@ -831,5 +831,5 @@
     <visual>
       <geometry>
-        <mesh filename="package://ur_description/meshes/ur5/visual/upperarm.dae"/>
+        <mesh filename="package://ur_description/meshes/ur5/visual/upperarm.stl"/>
       </geometry>
       <material name="LightGrey">
@@ -859,5 +859,5 @@
     <visual>
       <geometry>
-        <mesh filename="package://ur_description/meshes/ur5/visual/forearm.dae"/>
+        <mesh filename="package://ur_description/meshes/ur5/visual/forearm.stl"/>
       </geometry>
       <material name="LightGrey">
@@ -887,5 +887,5 @@
     <visual>
       <geometry>
-        <mesh filename="package://ur_description/meshes/ur5/visual/wrist1.dae"/>
+        <mesh filename="package://ur_description/meshes/ur5/visual/wrist1.stl"/>
       </geometry>
       <material name="LightGrey">
@@ -915,5 +915,5 @@
     <visual>
       <geometry>
-        <mesh filename="package://ur_description/meshes/ur5/visual/wrist2.dae"/>
+        <mesh filename="package://ur_description/meshes/ur5/visual/wrist2.stl"/>
       </geometry>
       <material name="LightGrey">
@@ -943,5 +943,5 @@
     <visual>
       <geometry>
-        <mesh filename="package://ur_description/meshes/ur5/visual/wrist3.dae"/>
+        <mesh filename="package://ur_description/meshes/ur5/visual/wrist3.stl"/>
       </geometry>
       <material name="LightGrey">
@@ -1057,5 +1057,5 @@
       <geometry>
         <!-- Origin of this mesh is the focal point of the LIDAR. -->
-        <mesh filename="package://lms1xx/meshes/sick-lms1xx.dae"/>
+        <mesh filename="package://lms1xx/meshes/sick-lms1xx.stl"/>
       </geometry>
     </visual>
@@ -1110,5 +1110,5 @@
       <origin rpy="-1.5707 0 -1.5707" xyz="0 0 0"/>
       <geometry>
-        <mesh filename="package://pointgrey_camera_description/meshes/pointgrey_bumblebee2.dae"/>
+        <mesh filename="package://pointgrey_camera_description/meshes/pointgrey_bumblebee2.stl"/>
       </geometry>
     </visual>
@@ -1212,5 +1212,5 @@
       <origin rpy="0 0 0" xyz="0 0 0"/>
       <geometry>
-        <mesh filename="package://robotiq_force_torque_sensor/meshes/visual/robotiq_fts300.dae"/>
+        <mesh filename="package://robotiq_force_torque_sensor/meshes/visual/robotiq_fts300.stl"/>
       </geometry>
       <material name="black"/>
@@ -1219,5 +1219,5 @@
       <origin rpy="0 0 0" xyz="0 0 0"/>
       <geometry>
-        <mesh filename="package://robotiq_force_torque_sensor/meshes/collision/robotiq_fts300.dae"/>
+        <mesh filename="package://robotiq_force_torque_sensor/meshes/collision/robotiq_fts300.stl"/>
       </geometry>
     </collision>
@@ -1253,5 +1253,5 @@
       <origin rpy="0 0 0" xyz="0 0 0"/>
       <geometry>
-        <mesh filename="package://robotiq_force_torque_sensor/meshes/visual/robotiq_fts300.dae"/>
+        <mesh filename="package://robotiq_force_torque_sensor/meshes/visual/robotiq_fts300.stl"/>
       </geometry>
       <material name="black"/>
@@ -1260,5 +1260,5 @@
       <origin rpy="0 0 0" xyz="0 0 0"/>
       <geometry>
-        <mesh filename="package://robotiq_force_torque_sensor/meshes/collision/robotiq_fts300.dae"/>
+        <mesh filename="package://robotiq_force_torque_sensor/meshes/collision/robotiq_fts300.stl"/>
       </geometry>
     </collision>
